File: weather_station.sch (KiCad schematic (older format))
At the start: 20 parts, among them J1 Barrel_Jack, U1 L7805, U2 LD1117S33TR, U3 RTC-DS3231, U4 DHT11, U5 LCDHD44780-->I2C, U6 NRF24L01_Breakout, U7 ATmega328-PU, Y1 16Mhz

Commit message: Poprawiona płytka (konektor NRF24 oraz otwory na śrubki)
Parts:
- U6: footprint RF_Module:nRF24L01_Breakout -> weather_station:NRF24-horizontal-pin-socket
Changed lines of the file:
@@
 F 0 "U6" H 4700 5950 50  0000 L CNN
 F 1 "NRF24L01_Breakout" H 4250 5750 50  0000 L CNN
-F 2 "RF_Module:nRF24L01_Breakout" H 6050 6350 50  0001 L CIN
+F 2 "weather_station:NRF24-horizontal-pin-socket" H 6050 6350 50  0001 L CIN
 F 3 "http://www.nordicsemi.com/eng/content/download/2730/34105/file/nRF24L01_Product_Specification_v2_0.pdf" H 5900 5650 50  0001 C CNN
 	1    5900 5750
